File: FT232H.sch (KiCad schematic (older format))
At the start: 25 parts, among them J1 USB_B_Micro, J2 Conn_01x10_Male, J3 Conn_01x10_Male, U1 93LC56B, U2 FT232H, Y1 12MHz

Commit message: Add PCB layout
Parts:
- removed J2, J3: Conn_01x10_Male, symbol Connector:Conn_01x10_Male
- added J2, J3: Conn_01x10, Connector_PinHeader_2.54mm:PinHeader_1x10_P2.54mm_Vertical, symbol Connector_Generic:Conn_01x10
- C1, C2, C3, C4, C5, C6, C7, C8: symbol device:C_Small -> FT232H-rescue:C_Small-device
- D1, D2: footprint LEDs:LED_0606 -> LED_SMD:LED_0603_1608Metric; symbol device:LED_Small -> FT232H-rescue:LED_Small-device
- J1: footprint Connectors:USB_Micro-B -> Connector_USB:USB_Micro-B_Molex_47346-0001
- L1, L2: symbol device:Ferrite_Bead_Small -> FT232H-rescue:Ferrite_Bead_Small-device
- R1, R2, R3, R4, R5, R6, R7: symbol device:R_Small -> FT232H-rescue:R_Small-device
- Y1: footprint Crystals:Resonator_SMD-3pin_7.2x3.0mm_HandSoldering -> Crystal:Resonator_SMD_muRata_CSTxExxV-3Pin_3.0x1.1mm; symbol device:Resonator -> FT232H-rescue:Resonator-device
Connections:
- wire segments 179 -> 189
- no-connect marks 2 -> 1

Commit message: Add BOM
Parts:
- C1, C2, C3, C4, C5, C6, C7, C8: symbol FT232H-rescue:C_Small-device -> Device:C_Small
- D1, D2: symbol FT232H-rescue:LED_Small-device -> Device:LED_Small
- L1, L2: symbol FT232H-rescue:Ferrite_Bead_Small-device -> Device:Ferrite_Bead_Small
- R1: value 17K -> 12K; symbol FT232H-rescue:R_Small-device -> Device:R_Small
- R2, R3, R4, R5, R6, R7: symbol FT232H-rescue:R_Small-device -> Device:R_Small
- Y1: symbol FT232H-rescue:Resonator-device -> Device:Resonator
Changed lines of the file:
@@
 $EndComp
 $Comp
-L FT232H-rescue:Resonator-device Y1
+L Device:Resonator Y1
 U 1 1 5BC5C351
 P 4500 3900
@@
 $EndComp
 $Comp
-L FT232H-rescue:R_Small-device R5
+L Device:R_Small R5
 U 1 1 5BC5CD62
 P 3150 4100
@@
 	5000 4150 5000 4300
 $Comp
-L FT232H-rescue:R_Small-device R2
+L Device:R_Small R2
 U 1 1 5BC5D91B
 P 4850 3250
@@
 	5850 4700 5950 4700
 $Comp
-L FT232H-rescue:C_Small-device C5
+L Device:C_Small C5
 U 1 1 5BC68289
 P 3150 5200
@@
 $EndComp
 $Comp
-L FT232H-rescue:C_Small-device C6
+L Device:C_Small C6
 U 1 1 5BC682CC
 P 3450 5200
@@
 $EndComp
 $Comp
-L FT232H-rescue:C_Small-device C7
+L Device:C_Small C7
 U 1 1 5BC682F2
 P 3700 5200
@@
 	6100 1900 6200 1900
 $Comp
-L FT232H-rescue:C_Small-device C3
+L Device:C_Small C3
 U 1 1 5BC7272A
 P 5500 1650
@@
 $EndComp
 $Comp
-L FT232H-rescue:C_Small-device C4
+L Device:C_Small C4
 U 1 1 5BC7276E
 P 6400 1650
@@
 $EndComp
 $Comp
-L FT232H-rescue:Ferrite_Bead_Small-device L2
+L Device:Ferrite_Bead_Small L2
 U 1 1 5BC7D1F2
 P 6750 1500
@@
 $EndComp
 $Comp
-L FT232H-rescue:Ferrite_Bead_Small-device L1
+L Device:Ferrite_Bead_Small L1
 U 1 1 5BC7D249
 P 5250 1500
@@
 $EndComp
 $Comp
-L FT232H-rescue:C_Small-device C1
+L Device:C_Small C1
 U 1 1 5BC8A11B
 P 2800 2050
@@
 $EndComp
 $Comp
-L FT232H-rescue:LED_Small-device D1
+L Device:LED_Small D1
 U 1 1 5BC9383F
 P 7200 4450
@@
 $EndComp
 $Comp
-L FT232H-rescue:LED_Small-device D2
+L Device:LED_Small D2
 U 1 1 5BC938CC
 P 7600 4450
@@
 $EndComp
 $Comp
-L FT232H-rescue:R_Small-device R3
+L Device:R_Small R3
 U 1 1 5BC93906
 P 7200 4750
@@
 $EndComp
 $Comp
-L FT232H-rescue:R_Small-device R4
+L Device:R_Small R4
 U 1 1 5BC9397F
 P 7600 4750
@@
 	7600 4850 7600 4950
 $Comp
-L FT232H-rescue:R_Small-device R6
+L Device:R_Small R6
 U 1 1 5BCA3B6A
 P 8250 4600
@@
 $EndComp
 $Comp
-L FT232H-rescue:R_Small-device R7
+L Device:R_Small R7
 U 1 1 5BCA3BC0
 P 8250 4900
@@
 $EndComp
 $Comp
-L FT232H-rescue:C_Small-device C8
+L Device:C_Small C8
 U 1 1 5BCB2F58
 P 4100 2350
@@
 	5100 2550 4950 2550
 $Comp
-L FT232H-rescue:C_Small-device C2
+L Device:C_Small C2
 U 1 1 5BCC0981
 P 4850 2550
@@
 $EndComp
 $Comp
-L FT232H-rescue:R_Small-device R1
+L Device:R_Small R1
 U 1 1 5BCC25BD
 P 4250 3050
 F 0 "R1" V 4150 3050 50  0000 C CNN
-F 1 "17K" V 4350 3050 50  0000 C CNN
+F 1 "12K" V 4350 3050 50  0000 C CNN
 F 2 "Resistors_SMD:R_0603_HandSoldering" H 4250 3050 50  0001 C CNN
 F 3 "~" H 4250 3050 50  0001 C CNN
